File: NDTU/Tele board.kicad_sch (KiCad schematic)
At the start: 85 parts, among them J1 Conn_01x02, J2 USB_C_Receptacle_USB2.0_16P, J3 Micro_SD_Card, SW1 SW_Push, U1 STM32H573VITx, U10 TLV75533PDRV, U11 L89, U12 AMS1117, U2 BMP280, U3 MS5611-01BA, U4 BMI088, U5 MMC5983MA, U6 KX134-1211, U7 TPS565208, U8 TPS62162DSG, U9 E22-900M30S, Y1 Crystal_GND24

Commit message: Add files via upload
Parts:
- removed BT1: 7.4V, symbol Device:Battery
- removed SW1: SW_Push, symbol Switch:SW_Push
- removed U10: TLV75533PDRV, Package_SON:WSON-6-1EP_2x2mm_P0.65mm_EP1x1.6mm, symbol Regulator_Linear:TLV75533PDRV
- removed U11: L89, E22-900M30S:XCVR_E22-900M30S, symbol E22-900M30S:E22-900M30S
- removed U12: AMS1117, Package_TO_SOT_SMD:SOT-223-3_TabPin2, symbol Regulator_Linear:AMS1117
- removed U7: TPS565208, Package_TO_SOT_SMD:SOT-23-6, symbol Regulator_Switching:TPS565208
- removed U8: TPS62162DSG, Package_SON:WSON-8-1EP_2x2mm_P0.5mm_EP0.9x1.6mm_ThermalVias, symbol Regulator_Switching:TPS62162DSG
- removed Y1: Crystal_GND24, symbol Device:Crystal_GND24_Small
- added C40, C41, C43, C44: 47pF, Capacitor_SMD:C_0603_1608Metric, symbol Device:C_Small
- added C42: 4.7nF, Capacitor_SMD:C_0603_1608Metric, symbol Device:C_Small
- added C45: 1uF, Capacitor_SMD:C_0603_1608Metric, symbol Device:C_Small
- added C46: 100nF, Capacitor_SMD:C_0603_1608Metric, symbol Device:C_Small
- added D1: D_Schottky, Diode_SMD:D_SOD-128, symbol Device:D_Schottky
- added E1: LI0603G121R-10, NewLib:IND_LI0603G121R-10_LRD-M, symbol LI0603G121R-10:LI0603G121R-10
- added IC1: MPXV5100DP, NewLib:MPXV5100DP, symbol NewLib1:MPXV5100DP
- added J4, J5: Conn_01x02_Pin, Connector_JST:JST_EH_B2B-EH-A_1x02_P2.50mm_Vertical, symbol Connector:Conn_01x02_Pin
- added R24, R25: 60, Resistor_SMD:R_0603_1608Metric, symbol Device:R_Small
- added R26: 27, Resistor_SMD:R_0603_1608Metric, symbol Device:R_Small
- added R27: 100, Resistor_SMD:R_0603_1608Metric, symbol Device:R_Small
- added R28, R29: 4.7k, Resistor_SMD:R_0603_1608Metric, symbol Device:R_Small
- added R30: 20k, Resistor_SMD:R_0603_1608Metric, symbol Device:R_Small
- added R31, R32: 10k, Resistor_SMD:R_0603_1608Metric, symbol Device:R_Small
- added U10: AP63200WU, Package_TO_SOT_SMD:TSOT-23-6, symbol Regulator_Switching:AP63200WU
- added U13: TCAN332, Package_SO:SOIC-8_3.9x4.9mm_P1.27mm, symbol Interface_CAN_LIN:TCAN332
- added U14: ADS1115IDGS, Package_SO:TSSOP-10_3x3mm_P0.5mm, symbol Analog_ADC:ADS1115IDGS
- added U7: TPS62162DSG, Package_SON:Texas_DSG0008A_WSON-8-1EP_2x2mm_P0.5mm_EP0.9x1.6mm_ThermalVias, symbol Regulator_Switching:TPS62162DSG
- added U8: L89, NewLib:XCVR_L89, symbol NewLib1:L89
- added Y2: ABMM2-8MHz, NewLib:CRYSTAL_ABMM2_ABR, symbol NewLib1:ABMM2-8.000MHZ-D1-T
- BT2: value Battery_Cell -> 3.3V
- C32: value 10uF -> 100nF
- C33: value 10uF -> 1uF
- C34: value 100nF -> 10nF
- C36: value C_Small -> 100nF
- C37: value C_Small -> 4.7uF
- C38, C39: footprint Package_QFP:LQFP-100_14x14mm_P0.5mm -> Capacitor_SMD:C_0603_1608Metric
- C7: value 10nF -> 1uF
- J1: footprint (none) -> Connector_AMASS:AMASS_XT30U-M_1x02_P5.0mm_Vertical
- J2: footprint (none) -> Connector_USB:USB_C_Receptacle_GCT_USB4105-xx-A_16P_TopMnt_Horizontal
- J3: footprint Package_DFN_QFN:OnSemi_UDFN-16-1EP_1.35x3.3mm_P0.4mm_EP0.4x2.8mm -> Connector_Card:microSD_HC_Hirose_DM3AT-SF-PEJM5
- L1, L2: footprint (none) -> Inductor_SMD:L_Coilcraft_XAL4020-XXX
- R17: value 10k -> 27
- R19, R20, R21, R22, R23: footprint (none) -> Resistor_SMD:R_0603_1608Metric
- U5: footprint MMC5983MA:PQFN50P300X300X100-16N -> NewLib:PQFN50P300X300X100-16N
- U6: footprint (none) -> NewLib:LGA12_2X2X0P9_ROM-M
- U9: footprint E22-900M30S:XCVR_E22-900M30S -> NewLib:XCVR_E22-900M30S
Connections:
- net +3V3: now also U3.2 (PS), E1.1, R28.1, R29.1, R32.2, U13.3 (VCC), U14.8 (VDD), U7.6 (VOS), U8.4 (VCC); no longer C26.1, C28.1, C33.1, C34.1, U1.22 (VDDA), U9.10 (VCC), U9.9 (VCC)
- net +5V: now also C26.1, C28.1, C34.1, U9.10 (VCC), U9.9 (VCC), C45.1, IC1.2 (VS), U7.2 (VIN), U7.3 (EN); no longer C32.1, R17.1
- net BAT+: now also J1.2 (Pin_2), D1.2 (A); no longer C16.1, C17.1, C18.1, J1.1 (Pin_1), R18.1
- net GND: now also C32.2, J1.1 (Pin_1), C40.2, C41.2, C42.2, C43.2, C44.2, C45.2, C46.2, IC1.3 (GND), R30.2, U10.4 (GND), U13.2 (GND), U14.1 (ADDR), U14.3 (GND), U7.1 (PGND), U7.4 (AGND), U8.12 (GND), U8.3 (GND), Y2.2, Y2.4; no longer J1.2 (Pin_2), U3.2 (PS), U3.6 (SDO)
- net I2C1_SCL: no longer R15.1, R4.2, U3.8 (SCLK), U5.1 (SCL/SPI_SCK)
- net I2C1_SDA: no longer R16.1, R3.2, U3.7 (SDI/SDA), U5.16 (SDA/SPI_SDI)
- net PD0: no longer U9.14 (BUSY)
- net PD1: no longer U9.13 (DIO1)
- net PD3: no longer U9.15 (~{RST})
- net PD4: no longer U9.6 (RXEN)
- net PD5: no longer U9.7 (TXEN)
- net at C19.2, L1.1: now also U10.5 (SW)
- net at R10.1, R11.1: now also U10.1 (FB)
- net at C10.2, R7.1, U1.12 (PH0): now also Y2.1
- net at C11.1, R7.2, U1.13 (PH1): now also Y2.3
- net USB+: now reaches R17.2
- net USB+: now also U1.71 (PA12)
- net at C19.1: now also U10.6 (BST)
- net at R13.2, R14.1: now also U7.5 (FB)
- net at L2.1: now also U7.7 (SW)
- net at R12.2: now also U7.8 (PG)
- net PC0: now reaches U1.15 (PC0)
- net PC1: now reaches U1.16 (PC1)
- net PC2: now reaches U1.17 (PC2)
- net PC3: now reaches U1.18 (PC3)
- net PE3: now reaches U1.2 (PE3)
- net GNSS_RX: now reaches U1.23 (PA0)
- net GNSS_RX: now also U8.1 (RXD)
- net GNSS_TX: now reaches U1.24 (PA1)
- net GNSS_TX: now also U8.2 (TXD)
- net GNSS_WU: now reaches U1.25 (PA2)
- net GNSS_WU: now also R32.1, U8.7 (WAKE_UP)
- net PA3: now reaches U1.26 (PA3)
- net PA3: now also U8.10 (~{RESET})
- net PC4: now reaches U1.33 (PC4)
- net PC5: now reaches U1.34 (PC5)
- net PB0: now reaches U1.35 (PB0)
- net PB1: now reaches U1.36 (PB1)
- net PB2: now reaches U1.37 (PB2)
- net PB2: now also U9.15 (~{RST})
- net PE7: now reaches U1.38 (PE7)
- net PE7: now also U9.14 (BUSY)
- net PE8: now reaches U1.39 (PE8)
- net PE8: now also U9.13 (DIO1)
- net PE9: now reaches U1.40 (PE9)
- net PE9: now also U9.6 (RXEN)
- net PE10: now reaches U1.41 (PE10)
- net PE10: now also U9.7 (TXEN)
- net PE15: now reaches U1.46 (PE15)
- net PB10: now reaches U1.47 (PB10)
- net PD8: now reaches U1.55 (PD8)
- net PD9: now reaches U1.56 (PD9)
- net PD10: now reaches U1.57 (PD10)
- net CAN_TX: now reaches U1.58 (PD11)
- net CAN_TX: now also U13.1 (TXD)
- net CAN_RX: now reaches U1.59 (PD12)
- net CAN_RX: now also U13.4 (RXD)
- net PD13: now reaches U1.60 (PD13)
- net PD14: now reaches U1.61 (PD14)
- net PD15: now reaches U1.62 (PD15)
- net PC6: now reaches U1.63 (PC6)
- net PC7: now reaches U1.64 (PC7)
- net PC8: now reaches U1.65 (PC8)
- net PC9: now reaches U1.66 (PC9)
- net PA8: now reaches U1.67 (PA8)
- net PA9: now reaches U1.68 (PA9)
- net PA10: now reaches U1.69 (PA10)
- net PC13: now reaches U1.7 (PC13)
- net PA13(JTMS: now reaches U1.72 (PA13(JTMS)
- net PA14(JTCK: now reaches U1.76 (PA14(JTCK)
- net PA15(JTDI): now reaches U1.77 (PA15(JTDI))
- net PC14: now reaches U1.8 (PC14)
- net PB3(JTDO: now reaches U1.89 (PB3(JTDO)
- net PC15: now reaches U1.9 (PC15)
- net PB4(NJTRST): now reaches U1.90 (PB4(NJTRST))
- net I2C4_SMBA: now reaches U1.91 (PB5)
- net I2C4_SCL: now reaches U1.92 (PB6)
- net I2C4_SCL: now also R15.1, R4.2, U3.8 (SCLK), U5.1 (SCL/SPI_SCK), R28.2, U14.10 (SCL)
- net I2C4_SDA: now reaches U1.93 (PB7)
- net I2C4_SDA: now also R16.1, R3.2, U3.7 (SDI/SDA), U5.16 (SDA/SPI_SDI), R29.2, U14.9 (SDA)
- net PE0: now reaches U1.97 (PE0)
- net at BT2.1 (+), C36.1, C37.1: now also U8.5 (V_BCKP)
- net at R18.2: now also U10.2 (EN)
- net USB_DM renamed D-
- net D-: now also R26.1; no longer U1.70 (PA11)
- net USB_DP renamed D+
- net D+: now also R17.1; no longer U1.71 (PA12)
- new net: C32.1, C33.1, E1.2, U1.22 (VDDA)
- new net: C42.1, R24.1, R25.1
- new net: C46.1, R31.2, U14.7 (AIN3)
- new net: IC1.4 (VOUT), R27.1
- new net AIN3: R27.2, R30.1, R31.1
- new net CAN+: C40.1, C43.1, J4.2 (Pin_2), J5.2 (Pin_2), R24.2, U13.7 (CANH)
- new net CAN-: C41.1, C44.1, J4.1 (Pin_1), J5.1 (Pin_1), R25.2, U13.6 (CANL)
- new net USB-: R26.2, U1.70 (PA11)
- new net V_IN: C16.1, C17.1, C18.1, D1.1 (K), R18.1, U10.3 (IN)
- no-connect marks 10 -> 33
Other:
- note added: "5V to 3.3V Buck Converter"
- note added: "ADS for Gauge"
- note added: "CAN Tranceiver"
- note added: "Differential Gauge"
- note removed: "5V to 3.3V LDO"
- moved on the sheet: C1, C10, C11, C19, C2, J1, J2, R1, R2, R7, R8, R9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

Commit message: Add files via upload
Parts:
- added C47: 100nF, Capacitor_SMD:C_0603_1608Metric, symbol Device:C_Small_US
- added J10, J11, J6, J7, J9: Conn_01x02, Connector_JST:JST_EH_B2B-EH-A_1x02_P2.50mm_Vertical, symbol Connector_Generic:Conn_01x02
- added Q1, Q2: SISA96DN-T1-GE3, NewLib:SIS862DNT1GE3, symbol SiSA96DN-T1:SISA96DN-T1-GE3
- added R33: 32.4k, Resistor_SMD:R_0603_1608Metric, symbol Device:R_Small
- added R34, R39: 42.2k, Resistor_SMD:R_0603_1608Metric, symbol Device:R_Small
- added R35, R36, R37: 10k, Resistor_SMD:R_0603_1608Metric, symbol Device:R_Small
- added R38: 80k, Resistor_SMD:R_0603_1608Metric, symbol Device:R_Small
- added R40, R42: 1k, Resistor_SMD:R_0603_1608Metric, symbol Device:R_Small
- added R41, R43: 33k, Resistor_SMD:R_0603_1608Metric, symbol Device:R_Small
- added U15: TPS2121RUXR, NewLib:IC_TPS2121RUXR, symbol TPS2121:TPS2121RUXR
Connections:
- net +5V: now also J10.1 (Pin_1), J11.1 (Pin_1), J6.1 (Pin_1), J7.1 (Pin_1), J9.1 (Pin_1), U15.1 (OUT), U15.8 (OUT); no longer C20.1, C21.1, C22.1, J2.A4 (VBUS), J2.A9 (VBUS), J2.B4 (VBUS), J2.B9 (VBUS), L1.2, R10.2
- net GND: now also C47.1, J10.2 (Pin_2), J11.2 (Pin_2), J9.2 (Pin_2), Q1.1 (S), Q1.2 (S), Q1.3 (S), Q2.1 (S), Q2.2 (S), Q2.3 (S), R35.1, R36.1, R37.1, R38.2, R41.1, R43.1, U15.12 (GND), U15.6 (PR1)
- new net: R33.2, R35.2, U15.3 (CP2)
- new net: R37.2, R39.2, U15.5 (OV1)
- new net: R38.1, U15.10 (ILM)
- new net: C47.2, U15.11 (SS)
- new net: R34.2, R36.2, U15.4 (OV2)
- new net BATT_5V: C20.1, C21.1, C22.1, L1.2, R10.2, R39.1, U15.7 (IN1)
- new net CAM: R40.1
- new net CAM2: R42.1
- new net CAM2_GND: J7.2 (Pin_2), Q2.5 (D), Q2.6 (D), Q2.7 (D), Q2.8 (D)
- new net CAM_GND: J6.2 (Pin_2), Q1.5 (D), Q1.6 (D), Q1.7 (D), Q1.8 (D)
- new net G_DROGUE: Q1.4 (G), R40.2, R41.2
- new net G_MAIN: Q2.4 (G), R42.2, R43.2
- new net USB_5V: J2.A4 (VBUS), J2.A9 (VBUS), J2.B4 (VBUS), J2.B9 (VBUS), R33.1, R34.1, U15.2 (IN2)
- no-connect marks 33 -> 34

Commit message: Add files via upload
Connections:
- net 3V3 is gone; now on net +3V3: U3.4 (CSB), U3.5 (CSB)
